File: radler.kicad_pcb (KiCad board)
At the start: 2 copper layers, 193 parts, among them J1 USB_B_Mini, SW1 Pause, SW10 F6, SW11 F7, SW12 F8, SW13 F9, SW14 F10, SW15 F11, SW16 F12, SW17 PgUp, SW18 Home, SW19 Ins, SW2 ScrLk, SW20 Backtick, SW21 1, SW22 2, SW23 3, SW24 4, SW25 5, SW26 6, SW27 7, SW28 8, SW29 9, SW3 PrtSc, SW30 0, SW31 -, SW32 =, SW33 Backspace, SW34 PgDn, SW35 End, SW36 Del, SW37 Tab, SW38 Q, SW39 W, SW4 Esc, SW40 E, SW41 R, SW42 T, SW43 Y, SW44 U, SW45 I, SW46 O, SW47 P, SW48 [, SW49 ], SW5 F1, SW50 \, SW51 CapsLock, SW52 A, SW53 S, SW54 D, SW55 F, SW56 G, SW57 H, SW58 J, SW59 K, SW6 F2, SW60 L, SW61 ;, SW62 ', SW63 Enter, SW64 Up, SW65 Shift, SW66 Z, SW67 X, SW68 C, SW69 V, SW7 F3, SW70 B, SW71 N, SW72 M, SW73 ,, SW74 ., SW75 /, SW76 RShift, SW77 Left, SW78 Down, SW79 Right, SW8 F4, SW80 Ctrl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

Commit message: organize pcb and schematic
Parts:
- removed SW88: RESET, Button_Switch_THT:SW_PUSH_6mm
- added LED0: A, LED_THT:LED_D3.0mm, F.Cu at (100.0, 19.1)
- added LED3: D, LED_THT:LED_D3.0mm, F.Cu at (107.0, 26.2)
- added R6: 1.5k, Resistor_THT:R_Axial_DIN0204_L3.6mm_D1.6mm_P7.62mm_Horizontal, F.Cu at (92.9, 23.8)
- added R7: 1.5k, Resistor_THT:R_Axial_DIN0204_L3.6mm_D1.6mm_P7.62mm_Horizontal, F.Cu at (92.9, 26.2)
- added RESET: RESET, Button_Switch_THT:SW_PUSH_6mm, F.Cu at (116.7, 21.4)
- D1, D10, D11, D12, D13, D14, D15, D16, D17, D18, D19, D2, D20, D21, D22, D23, D24, D25, D26, D27, D28, D29, D3, D30, D31, D32, D33, D34, D35, D36, D37, D38, D39, D4, D40, D41, D42, D43, D44, D45, D46, D47, D48, D49, D5, D50, D51, D52, D53, D54, D55, D56, D57, D58, D59, D6, D60, D61, D62, D63, D64, D65, D66, D67, D68, D69, D7, D70, D71, D72, D73, D74, D75, D76, D77, D78, D79, D8, D80, D81, D82, D83, D84, D85, D86, D87, D88, D89, D9: footprint Diode_THT:D_DO-35_SOD27_P5.08mm_Vertical_AnodeUp -> Diode_THT:D_DO-35_SOD27_P7.62mm_Horizontal
- J1: footprint keyboard_parts:USB_miniB -> Connector_USB:USB_B_OST_USB-B1HSxx_Horizontal
- LED1: value RED -> B
- LED2: value GREEN -> C
- R1: footprint Resistor_THT:R_Axial_DIN0204_L3.6mm_D1.6mm_P5.08mm_Horizontal -> Resistor_THT:R_Axial_DIN0204_L3.6mm_D1.6mm_P7.62mm_Horizontal
- R2: value R_Small -> 68; footprint Resistor_THT:R_Axial_DIN0204_L3.6mm_D1.6mm_P5.08mm_Horizontal -> Resistor_THT:R_Axial_DIN0204_L3.6mm_D1.6mm_P7.62mm_Horizontal
- R3: value 75 -> 68; footprint Resistor_THT:R_Axial_DIN0204_L3.6mm_D1.6mm_P5.08mm_Horizontal -> Resistor_THT:R_Axial_DIN0204_L3.6mm_D1.6mm_P7.62mm_Horizontal
- R4: value 75 -> 1.5k; footprint Resistor_THT:R_Axial_DIN0204_L3.6mm_D1.6mm_P5.08mm_Horizontal -> Resistor_THT:R_Axial_DIN0204_L3.6mm_D1.6mm_P7.62mm_Horizontal
- R5: value R_Small -> 1.5k; footprint Resistor_THT:R_Axial_DIN0204_L3.6mm_D1.6mm_P5.08mm_Horizontal -> Resistor_THT:R_Axial_DIN0204_L3.6mm_D1.6mm_P7.62mm_Horizontal
- SW20: value Backtick -> `
- SW65: value Shift -> LShift
- Y1: footprint Crystal:Crystal_HC49-U_Vertical -> Crystal:Crystal_HC49-4H_Vertical
- moved D16 374.5 mm to (361.9, 19.1), turned to 270 degrees
- moved D63 370.4 mm to (350.0, 11.9), turned to 270 degrees
- moved D50 336.3 mm to (357.2, 14.3), turned to 270 degrees
- moved D49 329.2 mm to (338.1, 14.3), turned to 270 degrees
- moved D61 324.8 mm to (319.1, 11.9), turned to 270 degrees
- moved SW63 319.0 mm to (352.4, 104.8)
- moved SW76 317.9 mm to (347.7, 123.8)
- moved D48 315.9 mm to (331.0, 14.3), turned to 270 degrees
- moved D60 314.6 mm to (304.8, 11.9), turned to 270 degrees
- moved D87 314.0 mm to (354.8, 7.14), turned to 270 degrees
- moved D72 313.4 mm to (276.2, 9.53), turned to 270 degrees
- moved D59 311.9 mm to (290.5, 11.9), turned to 270 degrees
- moved SW86 311.7 mm to (338.1, 142.9)
- moved D71 307.7 mm to (266.7, 9.53), turned to 270 degrees
- moved SW50 300.6 mm to (359.6, 85.7)
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Connections:
- J1 pad 4: Net-(J1-Pad4) -> GND
- J1 pad 5: GND -> Net-(J1-Pad5)
- R2 pad 1: Net-(LED1-Pad2) -> Net-(D88-Pad1)
- R2 pad 2: Net-(JP1-Pad2) -> USB_D+
- R3 pad 1: Net-(D88-Pad1) -> USB_D-
- R3 pad 2: USB_D+ -> Net-(D89-Pad1)
- R4 pad 1: USB_D- -> Net-(LED0-Pad2)
- R4 pad 2: Net-(D89-Pad1) -> LED0
- R5 pad 1: Net-(LED2-Pad2) -> Net-(LED1-Pad2)
- R5 pad 2: Net-(JP2-Pad2) -> LED1
- SW63 pad 2: Net-(SW63-Pad2) -> COL16
- SW76 pad 2: Net-(SW63-Pad2) -> COL16
- SW86 pad 2: Net-(SW63-Pad2) -> COL16
- U1 pad 1: COL2 -> COL17
- U1 pad 14: COL14 -> COL9
- U1 pad 15: COL15 -> COL8
- U1 pad 16: COL16 -> COL7
- U1 pad 17: COL17 -> COL6
- U1 pad 18: Net-(U1-Pad18) -> COL5
- U1 pad 19: Net-(U1-Pad19) -> COL4
- U1 pad 2: COL3 -> COL16
- U1 pad 20: Net-(U1-Pad20) -> COL3
- U1 pad 21: Net-(U1-Pad21) -> COL0
- U1 pad 22: i2c_SCL -> COL1
- U1 pad 23: i2c_SDA -> COL2
- U1 pad 24: USB_D- -> ROW0
- U1 pad 25: USB_D+ -> ROW1
- U1 pad 26: COL10 -> ROW2
- U1 pad 27: COL11 -> ROW3
- U1 pad 28: COL12 -> ROW4
- U1 pad 29: COL13 -> ROW5
- U1 pad 3: COL4 -> COL15
- U1 pad 33: COL1 -> Net-(U1-Pad33)
- U1 pad 34: COL0 -> Net-(U1-Pad34)
- U1 pad 35: ROW5 -> LED3
- U1 pad 36: ROW4 -> LED2
- U1 pad 37: ROW3 -> LED1
- U1 pad 38: ROW2 -> LED0
- U1 pad 39: ROW1 -> USB_D+
- U1 pad 4: COL5 -> COL14
- U1 pad 40: ROW0 -> USB_D-
- U1 pad 5: COL6 -> COL13
- U1 pad 6: COL7 -> COL12
- U1 pad 7: COL8 -> COL11
- U1 pad 8: COL9 -> COL10
